File: OpenAmiga2000CoproAdapter.sch (KiCad schematic (older format))
At the start: 18 parts, among them CN1 A2000_COPRO_SLOT, P1 CONN_2, P10 CONN_1, P11 CONN_1, P12 CONN_1, P13 CONN_1, P14 CONN_1, P15 CONN_1, P2 CONN_2, P3 CONN_2, P4 CONN_2, P5 CONN_1, P6 CONN_1, P7 CONN_1, P8 CONN_1, P9 CONN_1, P99 OSHW_LOGO, U1 68000D

Commit message: Memory bank 1
Parts:
- removed P99: OSHW_LOGO, Symbol:OSHW-Logo_7.5x8mm_Copper, symbol conn:CONN_1
- P1, P2, P3, P4: symbol conn:CONN_2 -> OpenAmiga2000CoproAdapter-rescue:CONN_2-conn
- P10, P11, P12, P13, P14, P15, P5, P6, P7, P8, P9: symbol conn:CONN_1 -> OpenAmiga2000CoproAdapter-rescue:CONN_1-conn
- U1: symbol CPU_NXP_68000:68000D -> OpenAmiga2000CoproAdapter-rescue:68000D-CPU_NXP_68000
Connections:
- net labels added: a[1..23], d[0..15]
- wire segments 186 -> 191
- no-connect marks 1 -> 0
