File: OpenAmiga2000CoproAdapter.sch (KiCad schematic (older format))
At the start: 21 parts, among them CN1 A2000_COPRO_SLOT, P1 CONN_2, P10 CONN_1, P11 CONN_1, P12 CONN_1, P13 CONN_1, P14 CONN_1, P15 CONN_1, P2 CONN_2, P3 CONN_2, P4 CONN_2, P5 CONN_1, P6 CONN_1, P7 CONN_1, P8 CONN_1, P9 CONN_1, U1 68000D

Commit message: finish routing
Parts:
- added C10: 100nF, Capacitor_THT:C_Disc_D7.0mm_W2.5mm_P5.00mm, symbol device:C
- added U10: Spare, Package_DIP:DIP-14_W7.62mm, symbol 74:74HC00
- renumbered C10 to C101, C20 to C102, C30 to C103
Connections:
- net +5V: now also C10.1, U10.14 (VCC)
- net GND: now also C10.2, U10.7 (GND)
Changed lines of the file:
@@
 Connection ~ 3550 5920
 $Comp
-L device:CP C30
+L device:CP C103
 U 1 1 60C785AA
 P 650 7400
-F 0 "C30" H 768 7446 50  0000 L CNN
+F 0 "C103" H 768 7446 50  0000 L CNN
 F 1 "47uF" H 700 7300 50  0000 L CNN
 F 2 "Capacitor_THT:CP_Radial_D5.0mm_P2.50mm" H 688 7250 50  0001 C CNN
@@
 $EndComp
 $Comp
-L device:CP C20
+L device:CP C102
 U 1 1 60C796C0
 P 1350 7400
-F 0 "C20" H 1468 7446 50  0000 L CNN
+F 0 "C102" H 1468 7446 50  0000 L CNN
 F 1 "47uF" H 1400 7300 50  0000 L CNN
 F 2 "Capacitor_THT:CP_Radial_D5.0mm_P2.50mm" H 1388 7250 50  0001 C CNN
@@
 $EndComp
 $Comp
-L device:CP C10
+L device:CP C101
 U 1 1 60C79EDB
 P 1000 7400
-F 0 "C10" H 1118 7446 50  0000 L CNN
+F 0 "C101" H 1118 7446 50  0000 L CNN
 F 1 "47uF" H 1050 7300 50  0000 L CNN
 F 2 "Capacitor_THT:CP_Radial_D5.0mm_P2.50mm" H 1038 7250 50  0001 C CNN
@@
 	1350 7550 1700 7550
 Connection ~ 1350 7550
+$Comp
+L 74:74HC00 U10
+U 5 1 60601FDC
+P 1100 5650
+F 0 "U10" H 1050 5700 50  0000 L CNN
+F 1 "Spare" H 950 5600 50  0000 L CNN
+F 2 "Package_DIP:DIP-14_W7.62mm" H 1100 5650 50  0001 C CNN
+F 3 "http://www.ti.com/lit/gpn/sn74hc00" H 1100 5650 50  0001 C CNN
+	5    1100 5650
+	1    0    0    -1
+$EndComp
+$Comp
+L device:C C10
+U 1 1 6062C309
+P 1450 5650
+F 0 "C10" H 1565 5696 50  0000 L CNN
+F 1 "100nF" H 1565 5605 50  0000 L CNN
+F 2 "Capacitor_THT:C_Disc_D7.0mm_W2.5mm_P5.00mm" H 1488 5500 50  0001 C CNN
+F 3 "~" H 1450 5650 50  0001 C CNN
+	1    1450 5650
+	1    0    0    -1
+$EndComp
+Wire Wire Line
+	1100 6150 1450 6150
+Wire Wire Line
+	1450 6150 1450 5800
+Wire Wire Line
+	1100 5150 1450 5150
+Wire Wire Line
+	1450 5150 1450 5500
 Wire Bus Line
 	6500 5400 6500 6100
@@
 Wire Bus Line
 	5000 900  5000 3510
+$Comp
+L OpenAmiga2000CoproAdapter-rescue:+5V-power #PWR0116
+U 1 1 6065E404
+P 1100 5150
+F 0 "#PWR0116" H 1100 5000 50  0001 C CNN
+F 1 "+5V" H 1115 5323 50  0000 C CNN
+F 2 "" H 1100 5150 50  0001 C CNN
+F 3 "" H 1100 5150 50  0001 C CNN
+	1    1100 5150
+	1    0    0    -1
+$EndComp
+Connection ~ 1100 5150
+$Comp
+L OpenAmiga2000CoproAdapter-rescue:GND-power #PWR0142
+U 1 1 6065EB22
+P 1100 6150
+F 0 "#PWR0142" H 1100 5900 50  0001 C CNN
+F 1 "GND" H 1105 5977 50  0000 C CNN
+F 2 "" H 1100 6150 50  0001 C CNN
+F 3 "" H 1100 6150 50  0001 C CNN
+	1    1100 6150
+	1    0    0    -1
+$EndComp
+Connection ~ 1100 6150
 $EndSCHEMATC
