File: OpenAmiga2000CoproAdapter.sch (KiCad schematic (older format))
At the start: 23 parts, among them CN1 A2000_COPRO_SLOT, P1 CONN_2, P10 CONN_1, P11 CONN_1, P12 CONN_1, P13 CONN_1, P14 CONN_1, P15 CONN_1, P2 CONN_2, P3 CONN_2, P4 CONN_2, P5 CONN_1, P6 CONN_1, P7 CONN_1, P8 CONN_1, P9 CONN_1, U1 68000D, U10 Spare

Commit message: rom mirror
Parts:
- C101, C102, C103: symbol device:CP -> OpenAmiga2000CoproAdapter-rescue:CP-device
Changed lines of the file:
@@
 Connection ~ 3550 5920
 $Comp
-L device:CP C103
+L OpenAmiga2000CoproAdapter-rescue:CP-device C103
 U 1 1 60C785AA
 P 650 7400
@@
 $EndComp
 $Comp
-L device:CP C102
+L OpenAmiga2000CoproAdapter-rescue:CP-device C102
 U 1 1 60C796C0
 P 1350 7400
@@
 $EndComp
 $Comp
-L device:CP C101
+L OpenAmiga2000CoproAdapter-rescue:CP-device C101
 U 1 1 60C79EDB
 P 1000 7400
